File: HARDWARE/REV B/SINGLE/TH.kicad_pcb (KiCad board)
At the start: 2 copper layers, 68.6 x 53.1 mm, 83 parts, among them P1 USB_OTG, P2 ICSP, P3 CONN_01X08, P4 CONN_01X06, P6 CONN_01X10, P7 CONN_01X08, P8 BARREL_JACK, U1 AMS1117-ADJ, U2 ATMEGA32U4-M, Y1 8MHz

Commit message: updated license, added BOM, KiCad 5
Parts:
- P1: value USB_OTG -> USB MINI B
- P8: value BARREL_JACK -> Barrel_Jack_Switch
